File: Integral_Granite.sch (EAGLE design)
At the start: 34 parts, among them IC1 TB6643KQ, IC2 TB6643KQ, IC3 TB6643KQ, IC4 TB6643KQ, IC5 TLP785_GB,F_, IC6 TLP785_GB,F_, J1 S7B-PH-K-S_LF__SN_, J10 S2B-PH-K-S_LF__SN_, J11 BS3P-SHF-1AA__LF__SN_, J2 S7B-PH-K-S_LF__SN_, J3 BS2P-SHF-1AA__LF__SN_, J4 BS2P-SHF-1AA__LF__SN_, J5 BS2P-SHF-1AA__LF__SN_, J6 BS2P-SHF-1AA__LF__SN_, J7 BS2P-SHF-1AA__LF__SN_, J8 BS2P-SHF-1AA__LF__SN_, J9 S2B-PH-K-S_LF__SN_, Q1 2SK4017_Q_, Q2 2SK4017_Q_

Commit message: 修正した
Parts:
- removed BR1, BR2: SE50PAJ-M3_I, SE50PAJ-M3_I:SE50PAJ-M3_I
- added D1, D2: SE50PAJ-M3_I, SE50PAJ-M3_I:SE50PAJ-M3_I
- renumbered IC1 to A1, IC2 to A2, IC3 to B1, IC4 to B2, J1 to SIGA, J10 to VDD, J11 to VS, J2 to SIGB, J3 to A1M, J4 to A2M, J5 to B1M, J6 to B2M, J7 to VDRIB, J8 to VSOL, J9 to SIGC
Connections:
- removed net KICKER_SIGNAL: C1.2, Q2.GATE, R3.2, VR1.CCW, VR1.WIPER
- removed net N$28: C1.1, IC6.EMITTER, R8.2
- new net KICKISO: C1.1, IC6.EMITTER, R3.2, R8.2
- new net KICKSIG: C1.2, Q2.GATE, VR1.CCW, VR1.WIPER
- net +24V: now also D2.K
- net +3V3: now also D1.K
- net GND: no longer BR1.K, BR2.K
- net N$20: now also D1.A; no longer BR1.A
- net N$22: now also D2.A; no longer BR2.A

Commit message: initial commit
Parts:
- removed SIGA, SIGB: S7B-PH-K-S_LF__SN_, S7B-PH-K-S_LF__SN_:S7B-PH-K-S_LF__SN_
- added MIN: S8B-PH-K-S_LF__SN_, S8B-PH-K-S_LF__SN_:S8B-PH-K-S_LF__SN_
Connections:
- net GND: no longer SIGA.1, SIGA.4, SIGA.7, SIGB.1, SIGB.4, SIGB.7
- net N$1: now also MIN.5; no longer SIGA.2
- net N$2: now also MIN.6; no longer SIGA.3
- net N$3: now also MIN.7; no longer SIGA.5
- net N$4: now also MIN.8; no longer SIGA.6
- net N$5: now also MIN.1; no longer SIGB.2
- net N$6: now also MIN.2; no longer SIGB.3
- net N$7: now also MIN.3; no longer SIGB.5
- net N$8: now also MIN.4; no longer SIGB.6
